File: HardWare/v1.0.1/MC_G431C8/Driver.kicad_sch (KiCad schematic)
At the start: 43 parts, among them J5 Conn_01x03, Q2 NCE6080K, Q3 NCE6080K, Q4 NCE6080K, Q5 NCE6080K, Q6 NCE6080K, Q7 NCE6080K, U2 fd6288t

Commit message: 20240603 HardWare优化
Parts:
- removed Q2, Q3, Q4, Q5, Q6, Q7: NCE6080K, Package_TO_SOT_SMD:TO-252-2, symbol Device:Q_NMOS_GDS
- added C32: 1nF, Capacitor_SMD:C_0603_1608Metric, symbol Device:C_Small
- added C33, C34, C35, C36, C37, C38: NC, Capacitor_SMD:C_0603_1608Metric, symbol Device:C
- added Q2, Q3, Q4, Q5, Q6, Q8: ~, Package_DFN_QFN:DFN-8-1EP_6x5mm_P1.27mm_EP4x4mm, symbol User_Power:HYG025N06
- added R29: 0.01R, Resistor_SMD:R_2512_6332Metric, symbol Device:R_US
- added R35, R36: 4.7K, Resistor_SMD:R_0603_1608Metric, symbol Device:R_US
- added R37, R39, R45: 1K(1%), Resistor_SMD:R_0603_1608Metric, symbol Device:R_US
- added R38, R40, R46: 6.8K, Resistor_SMD:R_0603_1608Metric, symbol Device:R_US
- added R41, R43, R47: 4.7K(1%), Resistor_SMD:R_0603_1608Metric, symbol Device:R_US
- added R42, R44, R48: 0R, Resistor_SMD:R_0603_1608Metric, symbol Device:R_US
- added U3: LMV324I, Package_SO:SSOP-14_5.3x6.2mm_P0.65mm, symbol User_Sensor:LMV324IDT
- D2, D6, D7: value 1N589 -> 1N5819
- R26: value 10K(1%) -> 10k
- R28, R34: value 0.01R(1%) -> 0.01R
- R32: value 4.7K(1%) -> 4.7K
- R33: value 10K(1%) -> 10K
- U2: footprint (none) -> Package_SO:TSSOP-20_4.4x5mm_P0.4mm
Connections:
- net +24V: now also C31.1, Q2.1 (S), Q2.2 (S), Q2.3 (S), Q5.1 (S), Q5.2 (S), Q5.3 (S), Q8.1 (S), Q8.2 (S), Q8.3 (S)
- net GND: now also C31.2, R34.2, C32.2, C34.1, C36.1, C38.1, R36.2, R37.1, R39.1, R45.1, U3.11 (G)
- net U: now also C22.1, J5.3 (Pin_3), U2.18 (VS1), Q3.1 (S), Q3.2 (S), Q3.3 (S), Q8.5 (D), Q8.6 (D), Q8.7 (D), Q8.8 (D), Q8.9 (D)
- net U_CH: now also U2.19 (HO1)
- net V: now also C22.2, C23.1, D2.1 (K), J5.2 (Pin_2), U2.15 (VS2), U2.20 (VB1), Q2.5 (D), Q2.6 (D), Q2.7 (D), Q2.8 (D), Q2.9 (D), Q4.1 (S), Q4.2 (S), Q4.3 (S)
- net V_CH: now also D10.1 (K), U2.16 (HO2)
- net V_CHN: now also U2.10 (LO2)
- net W: now also C25.1, J5.1 (Pin_1), U2.12 (VS3), Q5.5 (D), Q5.6 (D), Q5.7 (D), Q5.8 (D), Q5.9 (D), Q6.1 (S), Q6.2 (S), Q6.3 (S)
- net W_CH: now also U2.13 (HO3)
- net W_CHN: now also U2.9 (LO3)
- net i_u: now also Q3.5 (D), Q3.6 (D), Q3.7 (D), Q3.8 (D), Q3.9 (D), R38.2, U3.3 (+)
- net i_v: now also R28.1, Q4.5 (D), Q4.6 (D), Q4.7 (D), Q4.8 (D), Q4.9 (D), R40.2, U3.9 (-)
- net i_w: now also R34.1, Q6.5 (D), Q6.6 (D), Q6.7 (D), Q6.8 (D), Q6.9 (D), R46.2, U3.6 (-)
- net at D9.2 (A), R20.1, R22.1: now also Q8.4 (G)
- net at D13.2 (A), R31.1, R33.1: now also Q6.4 (G)
- net at D10.2 (A), R24.1, R26.1: now also Q2.4 (G)
- net at R32.1: now also D12.2 (A), R30.1, Q5.4 (G)
- net at D8.2 (A), R19.1, R21.1: now also Q3.4 (G)
- net at D11.2 (A), R25.1, R27.1: now also Q4.4 (G)
- net U_CHN: now reaches D8.1 (K), R19.2
- net U_CHN: now also U2.11 (LO1)
- new net: C37.1, R45.2, R47.1, U3.5 (+)
- new net: C37.2, R47.2, R48.1, U3.7
- new net: C35.1, R37.2, R43.1, U3.10 (+)
- new net: C35.2, R43.2, R44.1, U3.8 (11)
- new net: R35.2, R36.1, U3.12 (+)
- new net: C33.1, R39.2, R41.1, U3.2 (-)
- new net: C33.2, R41.2, R42.1, U3.1
- new net: R29.2, U3.13 (-), U3.14 (D_O)
- new net +3V3: C32.1, R35.1, U3.4 (V)
- new net OP_I_U: C34.2, R42.2
- new net OP_I_V: C36.2, R44.2
- new net OP_I_W: C38.2, R48.2
- new net Vref: R29.1, R38.1, R40.1, R46.1
- no-connect marks 6 -> 0
Other:
- note added: "1.65V基准电压"
- moved on the sheet: C26, C27, C28, C29, C30, C31, D10, D11, D12, D13, D8, D9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
