File: HardWare/v1.0.1/MC_G431C8/MC_G431C8.kicad_pcb (KiCad board)
At the start: 2 copper layers, 100 x 50 mm, 158 parts, among them J1 Conn_01x02, J2 Conn_01x03, J3 Conn_01x04, J4 Conn_01x06, J5 Conn_01x03, J6 Conn_01x02, Q1 MMBT3904L, U1 STM32G431C8, U2 fd6288t, U3 LMV324I, U4 TL431DBZ, U5 SGM6232YPS8G, U6 AMS1117-3.3, U7 AMS1117-5.0, U8 AS5047D, U9 TJA1042T-3, Y1 32MHZ

Commit message: 20240615 PCB绘制结束
Parts:
- removed TP10, TP11, TP12, TP13, TP8, TP9: TestPoint_Alt, TestPoint:TestPoint_Pad_D1.0mm
- moved TP5 2.17 mm to (138.4, 95.6)
- moved TP6 2.08 mm to (140.3, 94.5)
- moved TP3 1.66 mm to (109.0, 76.3)
- moved J5 0.25 mm to (180.3, 63.3)
- moved J6 0.07 mm to (141.3, 106.5)
Routing:
- net +3V3: track 143.8 -> 256.5 mm, vias 9 -> 11
- net GND: track 40.4 -> 106.0 mm, vias 38 -> 150
- net Vref: track 15.0 -> 46.0 mm, vias 0 -> 2
- net /Driver/V: track 38.9 -> 64.1 mm
- net +3.3VADC: track 11.7 -> 33.9 mm, vias 2 -> 3
- net +5V: track 143.3 -> 122.8 mm, vias 9 -> 7
- net /Driver/W: track 68.5 -> 87.9 mm
- net /Driver/U: track 37.4 -> 54.9 mm
- net /Driver/i_u: track 29.5 -> 26.1 mm
- net Net-(D12-A): track 10.9 -> 10.00 mm
- net /ADC_VBUS: track 51.1 -> 50.4 mm
- net /OP_I_V: track 19.7 -> 19.0 mm
- net /OP_I_W: track 16.8 -> 17.4 mm
- net /LED_01: track 57.1 -> 56.9 mm, vias 4 -> 3
- added copper zone on In1.Cu, net GND
- added copper zone on In2.Cu, net GND
Other:
- copper layers 2 -> 4
