File: HardWare/v1.0.1/MC_G431C8/MC_G431C8.kicad_sch (KiCad schematic)
At the start: 41 parts, among them J2 Conn_01x03, J3 Conn_01x04, J4 Conn_01x06, J6 Conn_01x02, U1 STM32G431C8, U9 TJA1042T-3, Y1 32MHZ

Commit message: 20240610 硬件布局完成95%，软件增加速度环
Connections:
- net KEY_01: now also U1.3 (PC14); no longer U1.26 (PB12)
- net SPI1_CLK: now also J4.3 (Pin_3); no longer J4.2 (Pin_2)
- net SPI1_CS: now also J4.2 (Pin_2); no longer J4.5 (Pin_5)
- net SPI1_MISO: now also J4.4 (Pin_4); no longer J4.3 (Pin_3)
- net SPI1_MOSI: now also J4.5 (Pin_5); no longer J4.4 (Pin_4)
- net SWCLK: now also J3.2 (Pin_2); no longer J3.3 (Pin_3)
- net SWDIO: now also J3.3 (Pin_3); no longer J3.2 (Pin_2)
- net CAN_H renamed CAN_N
- net CAN_L renamed CAN_P
- net CAN_RX renamed CAN_+
- net CAN_TX renamed CAN_-
Changed lines of the file:
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@@
+	)
+	(no_connect
+		(at 170.18 88.9)
 	)
 	(no_connect
@@
 	)
 	(no_connect
-		(at 116.84 59.69)
-	)
-	(no_connect
 		(at 154.94 101.6)
 	)
@@
 	(wire
 		(pts
+			(xy 109.22 59.69) (xy 116.84 59.69)
+		)
+		(stroke
+			(width 0)
+			(type default)
+		)
+	)
+	(wire
+		(pts
 			(xy 86.36 172.72) (xy 86.36 173.99)
 		)
@@
 		(pts
 			(xy 43.18 171.45) (xy 43.18 172.72)
-		)
-		(stroke
-			(width 0)
-			(type default)
-		)
-	)
-	(wire
-		(pts
-			(xy 170.18 88.9) (xy 184.15 88.9)
 		)
 		(stroke
@@
 		)
 	)
-	(label "CAN_H"
+	(label "CAN_N"
 		(at 134.62 144.78 0)
 		(fields_autoplaced yes)
@@
 		)
 	)
-	(label "CAN_RX"
+	(label "CAN_+"
 		(at 87.63 144.78 180)
 		(fields_autoplaced yes)
@@
 	)
 	(label "KEY_01"
-		(at 184.15 88.9 0)
+		(at 109.22 59.69 180)
 		(fields_autoplaced yes)
 		(effects
@@
 				(color 255 42 40 1)
 			)
-			(justify left bottom)
-		)
-	)
-	(label "CAN_L"
+			(justify right bottom)
+		)
+	)
+	(label "CAN_P"
 		(at 134.62 149.86 0)
 		(fields_autoplaced yes)
@@
 	)
 	(label "SWCLK"
-		(at 33.02 92.71 180)
+		(at 33.02 95.25 180)
 		(fields_autoplaced yes)
 		(effects
@@
 	)
 	(label "SPI1_MOSI"
-		(at 30.48 116.84 0)
+		(at 30.48 119.38 0)
 		(fields_autoplaced yes)
 		(effects
@@
 	)
 	(label "SPI1_CS"
-		(at 30.48 119.38 0)
+		(at 30.48 111.76 0)
 		(fields_autoplaced yes)
 		(effects
@@
 	)
 	(label "SWDIO"
-		(at 33.02 95.25 180)
+		(at 33.02 92.71 180)
 		(fields_autoplaced yes)
 		(effects
@@
 		)
 	)
-	(label "CAN_RX"
+	(label "CAN_+"
 		(at 182.88 71.12 0)
 		(fields_autoplaced yes)
@@
 	)
 	(label "SPI1_CLK"
-		(at 30.48 111.76 0)
+		(at 30.48 114.3 0)
 		(fields_autoplaced yes)
 		(effects
@@
 		)
 	)
-	(label "CAN_TX"
+	(label "CAN_-"
 		(at 87.63 142.24 180)
 		(fields_autoplaced yes)
@@
 		)
 	)
-	(label "CAN_H"
+	(label "CAN_N"
 		(at 30.48 135.89 0)
 		(fields_autoplaced yes)
@@
 		)
 	)
-	(label "CAN_L"
+	(label "CAN_P"
 		(at 30.48 138.43 0)
 		(fields_autoplaced yes)
@@
 	)
 	(label "SPI1_MISO"
-		(at 30.48 114.3 0)
+		(at 30.48 116.84 0)
 		(fields_autoplaced yes)
 		(effects
@@
 		)
 	)
-	(label "CAN_TX"
+	(label "CAN_-"
 		(at 182.88 68.58 0)
 		(fields_autoplaced yes)

Commit message: 20240615 PCB绘制结束
Parts:
- removed TP10, TP11, TP12, TP13, TP8, TP9: TestPoint_Alt, TestPoint:TestPoint_Pad_D1.0mm, symbol Connector:TestPoint_Alt
